File: hardware/navien_latest.kicad_pcb (KiCad board)
At the start: 2 copper layers, 64.6 x 36.9 mm, 30 parts, among them J1 Conn_01x03_MountingPin, J2 Conn_01x02, J3 S6B-XH-SM4-TB, Q1 2n7002, U1 WeMos_D1_mini, U2 THVD1406DR, U3 LM7805_TO220

Commit message: doc: consolidate Navien 240 documentation (240A/240A2): add doc/240.md, update README, remove doc/240-a.md
Parts:
- D1: footprint BIVAR_PIPE:LED-ARRAY-SMD_4P-L1.6-W1.5-BL-FD-WITH-PIPE-2 -> LED_SMD:LED-ARRAY-SMD_4P-L1.6-W1.5-BL-FD
- D5: footprint BIVAR_PIPE:LED-ARRAY-SMD_4P-L1.6-W1.5-BL-FD-WITH-PIPE-1 -> LED_SMD:LED-ARRAY-SMD_4P-L1.6-W1.5-BL-FD
- moved REF3 0.66 mm to (133.8, 106.4)
- moved REF2 0.60 mm to (133.8, 77.5)
Routing:
- net GND: track 11.3 -> 10.7 mm
Changed lines of the file:
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@@
 		)
 	)
-	(footprint "BIVAR_PIPE:LED-ARRAY-SMD_4P-L1.6-W1.5-BL-FD-WITH-PIPE-1"
+	(footprint "LED_SMD:LED-ARRAY-SMD_4P-L1.6-W1.5-BL-FD"
 		(layer "F.Cu")
 		(at 77.632452 101.8052 180)
@@
 			(at 0 -1.843 180)
 			(layer "F.SilkS")
-			(hide yes)
 			(effects
 				(font
@@
 			)
 		)
-		(property "Footprint" "BIVAR_PIPE:LED-ARRAY-SMD_4P-L1.6-W1.5-BL-FD-WITH-PIPE-1"
+		(property "Footprint" "LED-ARRAY-SMD_4P-L1.6-W1.5-BL-FD"
 			(at 0 0 180)
 			(layer "F.Fab")
@@
 			)
 		)
-		(property "LCSC" "C601684"
-			(at 0 0 0)
-			(layer "F.SilkS")
-			(hide yes)
-			(effects
-				(font
-					(size 1.27 1.27)
-					(thickness 0.15)
-				)
-			)
-		)
 		(property ki_fp_filters "LED* LED_SMD:* LED_THT:*")
 		(sheetname "Root")
 		(sheetfile "navien.kicad_sch")
+		(attr exclude_from_bom)
 		(fp_line
 			(start -0.889 1.016)
@@
 			(layer "F.SilkS")
 		)
-		(fp_rect
-			(start -2 -2)
-			(end 2.1 2.1)
-			(stroke
-				(width 0.1)
-				(type default)
-			)
-			(fill none)
-			(layer "F.SilkS")
-		)
 		(fp_poly
 			(pts
@@
 			(layer "User.3")
 		)
-		(pad "" np_thru_hole circle
-			(at -2 -2 180)
-			(size 1.524 1.524)
-			(drill 0.762)
-			(layers "*.Mask")
-		)
-		(pad "" np_thru_hole circle
-			(at 2.1 2.1 180)
-			(size 1.524 1.524)
-			(drill 0.762)
-			(layers "*.Mask")
-		)
 		(pad "1" smd rect
 			(at -0.95 0.45 90)
@@
 			)
 		)
-		(property "LCSC" "C17661"
+		(property "LCSC" "C17408"
 			(at 0 0 0)
 			(layer "F.SilkS")
@@
 			)
 		)
-		(property "LCSC" "C17661"
+		(property "LCSC" "C17634"
 			(at 0 0 0)
 			(layer "F.SilkS")
@@
 			)
 		)
-		(property "LCSC" "C53134"
-			(at 0 0 0)
-			(layer "F.SilkS")
-			(hide yes)
-			(effects
-				(font
-					(size 1.27 1.27)
-					(thickness 0.15)
-				)
-			)
-		)
 		(property ki_fp_filters "CP_*")
 		(sheetname "Root")
@@
 	(footprint "MountingHole:MountingHole_2.2mm_M2"
 		(layer "F.Cu")
-		(at 133.132452 106.2552)
+		(at 133.782452 106.3552)
 		(descr "Mounting Hole 2.2mm, no annular, M2")
 		(tags "mounting hole 2.2mm no annular m2")
@@
 		)
 	)
-	(footprint "BIVAR_PIPE:LED-ARRAY-SMD_4P-L1.6-W1.5-BL-FD-WITH-PIPE-2"
+	(footprint "LED_SMD:LED-ARRAY-SMD_4P-L1.6-W1.5-BL-FD"
 		(layer "F.Cu")
 		(at 77.432452 87.2052)
@@
 			(at 0 -1.843 0)
 			(layer "F.SilkS")
-			(hide yes)
 			(effects
 				(font
@@
 		)
 		(property "Value" "LED_RKGB"
-			(at -7.35 0.75 0)
+			(at 0 1.843 0)
 			(layer "F.Fab")
 			(effects
@@
 			)
 		)
-		(property "Footprint" "BIVAR_PIPE:LED-ARRAY-SMD_4P-L1.6-W1.5-BL-FD-WITH-PIPE-2"
+		(property "Footprint" "LED-ARRAY-SMD_4P-L1.6-W1.5-BL-FD"
 			(at 0 0 0)
 			(layer "F.Fab")
@@
 			)
 		)
-		(property "LCSC" "C601684"
-			(at 0 0 0)
-			(layer "F.SilkS")
-			(hide yes)
-			(effects
-				(font
-					(size 1.27 1.27)
-					(thickness 0.15)
-				)
-			)
-		)
 		(property ki_fp_filters "LED* LED_SMD:* LED_THT:*")
 		(sheetname "Root")
 		(sheetfile "navien.kicad_sch")
+		(attr exclude_from_bom)
 		(fp_line
 			(start -0.889 -1.016)
@@
 			(layer "F.SilkS")
 		)
-		(fp_rect
-			(start -2 -2)
-			(end 2.1 2.1)
-			(stroke
-				(width 0.1)
-				(type default)
-			)
-			(fill none)
-			(layer "F.SilkS")
-		)
 		(fp_poly
 			(pts
@@
 			(layer "User.3")
 		)
-		(pad "" np_thru_hole circle
-			(at -2 2.1)
-			(size 1.524 1.524)
-			(drill 0.762)
-			(layers "*.Mask")
-		)
-		(pad "" np_thru_hole circle
-			(at 2.1 -2)
-			(size 1.524 1.524)
-			(drill 0.762)
-			(layers "*.Mask")
-		)
 		(pad "1" smd rect
 			(at -0.95 0.45 270)
@@
 			)
 		)
-		(property "LCSC" "C17661"
+		(property "LCSC" "C17634"
 			(at 0 0 0)
 			(layer "F.SilkS")
@@
 			)
 		)
-		(property "LCSC" "C17604"
+		(property "LCSC" "C17634"
 			(at 0 0 0)
 			(layer "F.SilkS")
@@
 		(tags "capacitor tantalum")
 		(property "Reference" "C2"
-			(at -0.05 -1.8 0)
+			(at -1.5 -1.8 0)
 			(layer "F.SilkS")
 			(effects
@@
 			)
 		)
-		(property "LCSC" "C53134"
-			(at 0 0 0)
-			(layer "F.SilkS")
-			(hide yes)
-			(effects
-				(font
-					(size 1.27 1.27)
-					(thickness 0.15)
-				)
-			)
-		)
 		(property ki_fp_filters "CP_*")
 		(sheetname "Root")
@@
 		(tags "capacitor handsolder")
 		(property "Reference" "C1"
-			(at -1.45 1.7 0)
+			(at -2.5 -1.2 0)
 			(layer "F.SilkS")
 			(effects
@@
 		(sheetname "Root")
 		(sheetfile "navien.kicad_sch")
-		(attr through_hole exclude_from_pos_files exclude_from_bom)
+		(attr through_hole)
 		(fp_line
 			(start -1.33 -1.33)
@@
 		(tags "resistor handsolder")
 		(property "Reference" "R9"
-			(at 0.0076 -1.6392 0)
+			(at 3.1844 -0.0508 0)
 			(layer "F.SilkS")
 			(effects
@@
 		)
 		(property "Value" "10k"
-			(at 2.7076 -1.6892 0)
+			(at 3.4892 1.3716 0)
 			(layer "F.Fab")
 			(effects
@@
 	(footprint "MountingHole:MountingHole_2.2mm_M2"
 		(layer "F.Cu")
-		(at 133.182452 77.4552)
+		(at 133.782452 77.4552)
 		(descr "Mounting Hole 2.2mm, no annular, M2")
 		(tags "mounting hole 2.2mm no annular m2")
@@
 			)
 		)
-		(property "LCSC" "C17661"
+		(property "LCSC" "C17408"
 			(at 0 0 0)
 			(layer "F.SilkS")
@@
 	)
 	(gr_text "JLCJLCJLCJLC"
-		(at 108.582452 107.4052 0)
+		(at 109.282452 109.6552 0)
 		(layer "F.SilkS")
 		(effects
@@
 	)
 	(gr_text "Navien rs485 \nController\nRev 005\nHT 1.1.2026"
-		(at 108.582452 105.8552 0)
+		(at 109.282452 106.9552 0)
 		(layer "F.SilkS")
 		(effects
@@
 		(layer "Dwgs.User")
 		(pts
-			(xy 133.182452 106.5552) (xy 136.8044 103.7336)
+			(xy 133.8072 106.3752) (xy 136.8044 103.7336)
 		)
 		(height 8.128)
 		(orientation 0)
-		(gr_text "3.6219 mm"
+		(gr_text "2.9972 mm"
 			(at 134.874 116.1796 0)
 			(layer "Dwgs.User")
@@
 		(layer "Dwgs.User")
 		(pts
-			(xy 136.8044 77.2668) (xy 133.182452 79.5552)
+			(xy 136.8044 77.2668) (xy 133.8072 79.9084)
 		)
 		(height -8.128)
 		(orientation 0)
-		(gr_text "3.6219 mm"
+		(gr_text "2.9972 mm"
 			(at 135.7376 67.4624 0)
 			(layer "Dwgs.User")
@@
 	)
 	(segment
-		(start 122.168052 104.648)
-		(end 125.927252 104.648)
-		(width 0.5)
-		(layer "F.Cu")
-		(net 2)
-	)
-	(segment
-		(start 77.782452 99.1552)
-		(end 77.782452 99.9552)
+		(start 78.582452 97.9552)
+		(end 78.582452 101.3552)
 		(width 0.25)
 		(layer "F.Cu")
@@
 	)
 	(segment
-		(start 76.782452 98.1552)
-		(end 77.782452 99.1552)
-		(width 0.25)
+		(start 124.301652 104.648)
+		(end 124.555652 104.902)
+		(width 0.5)
 		(layer "F.Cu")
 		(net 2)
 	)
 	(segment
-		(start 113.9698 92.075)
-		(end 115.51615 92.075)
+		(start 122.168052 104.648)
+		(end 124.301652 104.648)
 		(width 0.5)
 		(layer "F.Cu")
@@
 	)
 	(segment
-		(start 77.782452 99.9552)
-		(end 78.582452 100.7552)
-		(width 0.25)
+		(start 124.555652 104.902)
+		(end 126.181252 104.902)
+		(width 0.5)
 		(layer "F.Cu")
 		(net 2)
 	)
 	(segment
-		(start 125.927252 104.648)
-		(end 126.181252 104.902)
+		(start 113.9698 92.075)
+		(end 115.51615 92.075)
 		(width 0.5)
 		(layer "F.Cu")
@@
 		(net 2)
 	)
-	(segment
-		(start 78.582452 100.7552)
-		(end 78.582452 101.3552)
-		(width 0.25)
-		(layer "F.Cu")
-		(net 2)
-	)
 	(via blind
 		(at 76.482452 87.6552)
@@
 	)
 	(via blind
-		(at 76.782452 98.1552)
+		(at 78.582452 97.9552)
 		(size 0.8)
 		(drill 0.4)
@@
 	(segment
 		(start 122.168052 107.188)
-		(end 126.050352 107.188)
+		(end 124.301652 107.188)
 		(width 0.5)
 		(layer "F.Cu")
@@
 	)
 	(segment
+		(start 124.301652 107.188)
+		(end 124.534152 106.9555)
+		(width 0.5)
+		(layer "F.Cu")
+		(net 19)
+	)
+	(segment
 		(start 119.729652 107.188)
 		(end 122.168052 107.188)
@@
 	)
 	(segment
-		(start 126.050352 107.188)
+		(start 124.534152 106.9555)
 		(end 126.282852 106.9555)
 		(width 0.5)
