File: hardware/navien-backups/navien-2025-12-14_143355/navien.kicad_pcb (KiCad board)
At the start: 2 copper layers, 64.6 x 36.9 mm, 30 parts, among them J1 Conn_01x03_MountingPin, J2 Conn_01x02, J3 S6B-XH-SM4-TB, Q1 2n7002, U1 WeMos_D1_mini, U2 THVD1406DR, U3 LM7805_TO220

Commit message: doc: consolidate Navien 240 documentation (240A/240A2): add doc/240.md, update README, remove doc/240-a.md
Parts:
- removed J2: Conn_01x02, Connector_PinHeader_2.54mm:PinHeader_1x02_P2.54mm_Vertical
- C2, C3: footprint Capacitor_Tantalum_SMD:CP_EIA-3216-18_Kemet-A_Pad1.58x1.35mm_HandSolder -> Capacitor_SMD:C_0805_2012Metric_Pad1.18x1.45mm_HandSolder
- D1: footprint BIVAR_PIPE:LED-ARRAY-SMD_4P-L1.6-W1.5-BL-FD-WITH-PIPE-2 -> LED_SMD:LED-ARRAY-SMD_4P-L1.6-W1.5-BL-FD-WITH-PIPE-2
- D5: footprint BIVAR_PIPE:LED-ARRAY-SMD_4P-L1.6-W1.5-BL-FD-WITH-PIPE-1 -> LED_SMD:LED-ARRAY-SMD_4P-L1.6-W1.5-BL-FD-WITH-PIPE-1
- R11: value 3K -> 25
- R12: value 3K -> 100
- R6: value 3k -> 100
- R7: value 3k -> 25
- R8: value 2k -> 25
- moved C2 25.8 mm to (87.9, 84.2), turned to -90 degrees
- moved C1 24.4 mm to (90.6, 84.1), turned to -90 degrees
- moved R10 1.21 mm to (117.9, 79.5), turned to 180 degrees
- moved REF3 1.15 mm to (133.8, 107.2)
- moved REF4 0.83 mm to (75.3, 107.2)
- moved REF2 0.60 mm to (133.8, 77.5)
Routing:
- net +5V: track 99.9 -> 94.0 mm, vias 2 -> 3
- net Net-(U1-CS/D8): track 23.7 -> 19.8 mm, vias 0 -> 1
- net Net-(U1-MOSI/D7): track 19.8 -> 16.7 mm, vias 0 -> 1
- net Net-(Q1-S): track 47.3 -> 44.5 mm
- net Net-(U1-SDA/D2): track 5.90 -> 6.56 mm
- net GND: track 11.3 -> 10.7 mm, vias 13 -> 14
- net +3.3V: track 49.1 -> 49.6 mm
Other:
- board text added: "Navien rs485 Controller HT 2.17.2025, Rev 001"
- board text removed: "Navien rs485 Controller Rev 005 HT 1.1.2026"
